File: pcb/moduleDriver/moduleDriver.kicad_sch (KiCad schematic)
At the start: 40 parts, among them J1 UART_RL, J10 Sensor, J11 Power, J12 Power, J13 Neopixel, J2 UART_LR, J3 MOTOR, J4 MOTOR, J5 MOTOR, J6 MOTOR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

Commit message: Single thread
Parts:
- removed C4: 0.1uF, Capacitor_SMD:C_0603_1608Metric, symbol Device:C_Small
- removed H4: MountingHole, MountingHole:MountingHole_3.2mm_M3_ISO7380, symbol Mechanical:MountingHole
- removed J10, J7, J8, J9: Sensor, Connector_PinHeader_2.54mm:PinHeader_1x03_P2.54mm_Vertical, symbol Connector:Conn_01x03_Male
- removed J13: Neopixel, Connector_PinHeader_2.54mm:PinHeader_1x03_P2.54mm_Vertical, symbol Connector:Conn_01x03_Male
- removed U5: 74HCT2G04GV, Package_SO:SC-74-6_1.5x2.9mm_P0.95mm, symbol New_Library:74HCT2G04GV
- added J10: Sense D, Connector_JST:JST_XH_B2B-XH-A_1x02_P2.50mm_Vertical, symbol Connector:Conn_01x02_Pin
- added J7: Sense A, Connector_JST:JST_XH_B2B-XH-A_1x02_P2.50mm_Vertical, symbol Connector:Conn_01x02_Pin
- added J8: Sense B, Connector_JST:JST_XH_B2B-XH-A_1x02_P2.50mm_Vertical, symbol Connector:Conn_01x02_Pin
- added J9: Sense C, Connector_JST:JST_XH_B2B-XH-A_1x02_P2.50mm_Vertical, symbol Connector:Conn_01x02_Pin
- added SW1: RUN, Button_Switch_THT:SW_PUSH_6mm, symbol Switch:SW_Push
- C2, C3: footprint Capacitor_SMD:C_0603_1608Metric -> Capacitor_SMD:C_1206_3216Metric
- D1, D2: footprint LED_SMD:LED_0603_1608Metric -> LED_SMD:LED_1206_3216Metric
- J1, J2: footprint Connector_PinHeader_2.54mm:PinHeader_1x03_P2.54mm_Vertical -> Connector_JST:JST_XH_B3B-XH-A_1x03_P2.50mm_Vertical
- J11, J12: footprint Library:ScrewTerminal-5.08-2P -> Connector_Phoenix_MSTB:PhoenixContact_MSTBA_2,5_2-G_1x02_P5.00mm_Horizontal
- J3: value MOTOR -> MOTOR A; symbol Connector:Conn_01x05_Male -> Connector_Generic:Conn_01x05
- J4: value MOTOR -> MOTOR B; symbol Connector:Conn_01x05_Male -> Connector_Generic:Conn_01x05
- J5: value MOTOR -> MOTOR C; symbol Connector:Conn_01x05_Male -> Connector_Generic:Conn_01x05
- J6: value MOTOR -> MOTOR D; symbol Connector:Conn_01x05_Male -> Connector_Generic:Conn_01x05
- R1, R10, R2, R3, R4, R5, R7, R8, R9: footprint Resistor_SMD:R_0603_1608Metric -> Resistor_SMD:R_1206_3216Metric
- R11: value 470 -> 1.2k; footprint Resistor_SMD:R_0603_1608Metric -> Resistor_SMD:R_1206_3216Metric; LCSC# C23179 -> C22765
- R6: value 2.2k -> 1.2k; footprint Resistor_SMD:R_0603_1608Metric -> Resistor_SMD:R_1206_3216Metric; LCSC# C4190 -> C22765
- U3, U4: footprint Package_SO:SOP-18_7x12.5mm_P1.27mm -> Package_DIP:DIP-18_W7.62mm_Socket
Connections:
- net GND: now also J11.1 (Pin_1), J10.1 (Pin_1), J7.1 (Pin_1), J8.1 (Pin_1), J9.1 (Pin_1), SW1.2; no longer J12.2 (Pin_2)
- net MOTOR_A_PHASE_A: now also U3.18 (O1); no longer U3.15 (O4)
- net MOTOR_A_PHASE_B: now also U3.17 (O2); no longer U3.16 (O3)
- net MOTOR_A_PHASE_C: now also U3.16 (O3); no longer U3.17 (O2)
- net MOTOR_A_PHASE_D: now also U3.15 (O4); no longer U3.18 (O1)
- net MOTOR_C_PHASE_A_P: now also U2.9 (GPIO6); no longer U2.17 (GPIO13/RX0)
- net MOTOR_C_PHASE_B_P: now also U2.10 (GPIO7); no longer U2.16 (GPIO12/TX0)
- net MOTOR_C_PHASE_C_P: now also U2.11 (GPIO8/TX1); no longer U2.15 (GPIO11)
- net MOTOR_C_PHASE_D_P: now also U2.12 (GPIO9/RX1); no longer U2.14 (GPIO10)
- net MOTOR_D_PHASE_A: now also U4.14 (O5); no longer U4.11 (O8)
- net MOTOR_D_PHASE_A_P: now also U2.14 (GPIO10); no longer U2.12 (GPIO9/RX1)
- net MOTOR_D_PHASE_B: now also U4.13 (O6); no longer U4.12 (O7)
- net MOTOR_D_PHASE_B_P: now also U2.15 (GPIO11); no longer U2.11 (GPIO8/TX1)
- net MOTOR_D_PHASE_C: now also U4.12 (O7); no longer U4.13 (O6)
- net MOTOR_D_PHASE_C_P: now also U2.16 (GPIO12/TX0); no longer U2.10 (GPIO7)
- net MOTOR_D_PHASE_D: now also U4.11 (O8); no longer U4.14 (O5)
- net MOTOR_D_PHASE_D_P: now also U2.17 (GPIO13/RX0); no longer U2.9 (GPIO6)
- net SENSOR_A: now also U2.2 (GPIO1/RX0), J7.2 (Pin_2); no longer U2.19 (GPIO14)
- net SENSOR_B: now also J8.2 (Pin_2)
- net SENSOR_C: now also U2.19 (GPIO14), J9.2 (Pin_2); no longer U2.2 (GPIO1/RX0)
- net SENSOR_D: now also J10.2 (Pin_2)
- net at R11.1: now also R6.2
- net VCC: now reaches D5.2 (A), J11.2 (Pin_2)
- net VCC: now also J12.2 (Pin_2); no longer J11.1 (Pin_1)
- net at R11.2: now also D2.2 (A)
- net RUN: now reaches U2.30 (RUN)
- net RUN: now also SW1.1
- net NEOPIXEL: no longer names the net of U2.1 (GPIO0/TX0)
- no-connect marks 7 -> 6
Other:
- note added: "Microswitches"
- note removed: "HALL EFFECT SENSORS"
- note removed: "Neopixel"
- moved on the sheet: D2, J11, J12
